File: hl8548-boost.kicad_pcb (KiCad board)
At the start: 2 copper layers, 35 parts, among them J2 BARREL_JACK, M1 HL8548, P1 CONN_01X06, P2 CONN_01X02, Q1 MUN5211DW, Q2 MUN5211DW, U1 SN74LVC1T45DBVR, U2 SN74LVC1T45DBVR, U3 ATOM010050030052, U4 USBLC6-4, U5 TPS76333, U6 NCP3170

Commit message: Weekly commit
Parts:
- removed P2: CONN_01X02, Pin_Headers:Pin_Header_Straight_1x02
- added C10: 30pF, Capacitors_SMD:C_0603, F.Cu at (157.0, 81.3)
- added D3: ESD7471, Meshium:SOD-882, F.Cu at (153.2, 96.3)
- added J1: BARREL_JACK, Connect:BARREL_JACK, F.Cu at (165.5, 57.5)
- added R6: R, Resistors_SMD:R_0603, F.Cu at (163.8, 90.2)
- C1: value 1uF -> 22uF; footprint Capacitors_SMD:C_0603 -> Capacitors_SMD:C_1206
- C3: value 10uF -> 1.5nF
- C4: value 0.01uF -> 22uF; footprint Capacitors_SMD:C_0603 -> Capacitors_SMD:C_1206
- C5: value 30pF -> 22uF; footprint Capacitors_SMD:C_0603 -> Capacitors_SMD:C_1206
- C6, C7: value 22uF -> 1uF; footprint Capacitors_SMD:C_1206 -> Capacitors_SMD:C_0603
- C8: value 22uF -> 10uF; footprint Capacitors_SMD:C_1206 -> Capacitors_SMD:C_0603
- C9: value 1.5nF -> 0.01uF
- J2: value BARREL_JACK -> JP3; footprint Connect:BARREL_JACK -> Meshium:JP3
- L1: value BLM21PG221SN1D -> 3.3uH; footprint Capacitors_SMD:C_0805 -> Meshium:CDRH6D38NP
- L2: value 3.3uH -> BLM21PG221SN1D; footprint Meshium:CDRH6D38NP -> Capacitors_SMD:C_0805
- M1: footprint LGA-234 -> Meshium:LGA-234
- R1: value R -> 0
- R2: value R -> 12.1K
- R4: value 12.1K -> 15K
- R5: value 15K -> R
- S1: value IPEX-20279-001E-01 -> CONN_01X10; footprint Meshium:IPEX-20279-001E-01 -> Pin_Headers:Pin_Header_Straight_1x10
- S3: value CONN_01X10 -> CONN_01X03; footprint Pin_Headers:Pin_Header_Straight_1x10 -> Pin_Headers:Pin_Header_Straight_1x03
- S4: value CONN_01X03 -> IPEX-20279-001E-01; footprint Pin_Headers:Pin_Header_Straight_1x03 -> Meshium:IPEX-20279-001E-01
- U1: value SN74LVC1T45DBVR -> NCP3170; footprint Meshium:SOT23-6 -> Meshium:SOIC8
- U3: value ATOM010050030052 -> SN74LVC1T45DBVR; footprint Meshium:ATOM010050030052 -> Meshium:SOT23-6; moved to F.Cu
- U4: value USBLC6-4 -> ATOM010050030052; footprint Meshium:SOT23-6L -> Meshium:ATOM010050030052; moved to B.Cu
- U6: value NCP3170 -> USBLC6-4; footprint Meshium:SOIC8 -> Meshium:SOT23-6L
- moved R2 81.5 mm to (146.3, 51.7), turned to 0 degrees
- moved R1 77.1 mm to (134.4, 61.1), turned to 270 degrees
- moved S1 70.7 mm to (122.0, 72.0), turned to 0 degrees
- moved C3 56.8 mm to (143.3, 52.5), turned to 270 degrees
- moved S3 53.5 mm to (162.9, 67.6), turned to 90 degrees
- moved U4 52.5 mm to (122.2, 61.1)
- moved S2 47.8 mm to (168.0, 72.0)
- moved C5 46.9 mm to (156.7, 62.4), turned to 90 degrees
- moved J2 45.9 mm to (146.2, 96.9)
- moved C4 45.7 mm to (154.4, 62.4), turned to 90 degrees
- moved L1 44.1 mm to (146.4, 62.5), turned to 90 degrees
- moved C6 43.4 mm to (122.7, 58.5), turned to 90 degrees
- moved U1 35.4 mm to (151.5, 57.4), turned to 180 degrees
- moved C1 34.3 mm to (154.4, 57.7), turned to 270 degrees
- moved D2 34.1 mm to (167.8, 100.1), turned to 180 degrees
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Connections:
- C4 pad 1: Net-(C3-Pad1) -> Net-(C4-Pad1)
- C5 pad 1: Net-(C3-Pad1) -> Net-(C4-Pad1)
- C6 pad 1: Net-(C2-Pad1) -> Net-(C6-Pad1)
- C7 pad 1: Net-(C2-Pad1) -> Net-(C4-Pad1)
- C8 pad 1: Net-(C8-Pad1) -> Net-(C10-Pad1)
- C9 pad 1: Net-(C9-Pad1) -> Net-(C10-Pad1)
- D1 pad 1: Net-(C2-Pad1) -> Net-(C4-Pad1)
- D2 pad 1: Net-(C2-Pad1) -> Net-(C4-Pad1)
- J2 pad 1: Net-(C8-Pad1) -> Net-(J2-Pad1)
- J2 pad 2: GND -> Net-(A1-Pad2)
- J2 pad 3: GND -> Net-(D3-Pad2)
- L1 pad 1: Net-(C2-Pad1) -> Net-(L1-Pad1)
- L1 pad 2: Net-(C3-Pad1) -> Net-(C4-Pad1)
- L2 pad 1: Net-(L2-Pad1) -> Net-(C4-Pad1)
- L2 pad 2: Net-(C2-Pad1) -> Net-(C10-Pad1)
- M1 pad 167: (no net) -> GND
- M1 pad 168: (no net) -> GND
- M1 pad 169: (no net) -> GND
- M1 pad 170: (no net) -> GND
- M1 pad 171: (no net) -> GND
- M1 pad 172: (no net) -> GND
- M1 pad 173: (no net) -> GND
- M1 pad 174: (no net) -> GND
- M1 pad 175: (no net) -> GND
- M1 pad 176: (no net) -> GND
- M1 pad 177: (no net) -> GND
- M1 pad 178: (no net) -> GND
- M1 pad 179: (no net) -> GND
- M1 pad 180: (no net) -> GND
- M1 pad 181: (no net) -> GND
- M1 pad 182: (no net) -> GND
- M1 pad 183: (no net) -> GND
- M1 pad 184: (no net) -> GND
- M1 pad 185: (no net) -> GND
- M1 pad 186: (no net) -> GND
- M1 pad 187: (no net) -> GND
- M1 pad 188: (no net) -> GND
- M1 pad 189: (no net) -> GND
- M1 pad 190: (no net) -> GND
- M1 pad 191: (no net) -> GND
- M1 pad 192: (no net) -> GND
- M1 pad 193: (no net) -> GND
- M1 pad 194: (no net) -> GND
- M1 pad 195: (no net) -> GND
- M1 pad 196: (no net) -> GND
- M1 pad 197: (no net) -> GND
- M1 pad 198: (no net) -> GND
- M1 pad 199: (no net) -> GND
- M1 pad 200: (no net) -> GND
- M1 pad 201: (no net) -> GND
- M1 pad 202: (no net) -> GND
- M1 pad 203: (no net) -> GND
- M1 pad 204: (no net) -> GND
- M1 pad 205: (no net) -> GND
- M1 pad 206: (no net) -> GND
- M1 pad 207: (no net) -> GND
- M1 pad 208: (no net) -> GND
- M1 pad 209: (no net) -> GND
- M1 pad 210: (no net) -> GND
- M1 pad 211: (no net) -> GND
- M1 pad 212: (no net) -> GND
- M1 pad 213: (no net) -> GND
- M1 pad 214: (no net) -> GND
- M1 pad 215: (no net) -> GND
- M1 pad 216: (no net) -> GND
- M1 pad 217: (no net) -> GND
- M1 pad 218: (no net) -> GND
- M1 pad 219: (no net) -> GND
- M1 pad 220: (no net) -> GND
- M1 pad 221: (no net) -> GND
- M1 pad 222: (no net) -> GND
- M1 pad 223: (no net) -> GND
- M1 pad 224: (no net) -> GND
- M1 pad 225: (no net) -> GND
- M1 pad 226: (no net) -> GND
- M1 pad 227: (no net) -> GND
- M1 pad 228: (no net) -> GND
- M1 pad 229: (no net) -> GND
- M1 pad 230: (no net) -> GND
- M1 pad 231: (no net) -> GND
- M1 pad 232: (no net) -> GND
- M1 pad 233: (no net) -> GND
- M1 pad 234: (no net) -> GND
- M1 pad 235: GND -> (no net)
- M1 pad 26: Net-(M1-Pad26) -> Net-(C6-Pad1)
- M1 pad 49: Net-(J1-Pad2) -> Net-(J2-Pad1)
- M1 pad 61: Net-(C3-Pad1) -> Net-(C10-Pad1)
- M1 pad 62: Net-(C3-Pad1) -> Net-(C10-Pad1)
- M1 pad 63: Net-(C3-Pad1) -> Net-(C10-Pad1)
- P1 pad 1: Net-(M1-Pad26) -> Net-(C6-Pad1)
- Q2 pad 1: GND -> Net-(Q2-Pad1)
- Q2 pad 2: Net-(M1-Pad60) -> Net-(M1-Pad1)
- Q2 pad 3: GND -> Net-(Q2-Pad3)
- Q2 pad 4: Net-(Q2-Pad4) -> GND
- Q2 pad 5: Net-(M1-Pad1) -> Net-(M1-Pad60)
- Q2 pad 6: Net-(Q2-Pad6) -> GND
- R1 pad 1: Net-(D1-Pad2) -> Net-(C2-Pad1)
- R1 pad 2: Net-(Q2-Pad4) -> /VCC_LP
- R2 pad 1: Net-(D2-Pad2) -> Net-(C3-Pad1)
- R2 pad 2: Net-(Q2-Pad6) -> Net-(R2-Pad2)
- R3 pad 2: Net-(C2-Pad1) -> Net-(C4-Pad1)
- R4 pad 1: Net-(C9-Pad1) -> GND
- R4 pad 2: Net-(R4-Pad2) -> Net-(R3-Pad1)
- R5 pad 1: GND -> Net-(D1-Pad2)
- R5 pad 2: Net-(R3-Pad1) -> Net-(Q2-Pad1)
- S1 pad 1: Net-(J1-Pad1) -> /VCC_LP
- S1 pad 2: GND -> Net-(S1-Pad2)
- S1 pad 3: GND -> /RXD
- S2 pad 1: /VCC_LP -> GND
- S2 pad 3: /RXD -> Net-(S2-Pad3)
- S2 pad 4: /TXD -> Net-(S2-Pad4)
- S2 pad 6: /RES -> Net-(S2-Pad6)
- S2 pad 7: /PWR_ON -> Net-(S2-Pad7)
- S3 pad 1: Net-(S3-Pad1) -> GND
- S3 pad 2: Net-(S3-Pad2) -> Net-(C1-Pad1)
- S3 pad 3: Net-(S3-Pad3) -> GND
- S4 pad 1: GND -> Net-(D3-Pad2)
- S4 pad 2: Net-(C8-Pad1) -> GND
- U1 pad 1: /VCC_LP -> GND
- U1 pad 2: GND -> Net-(C1-Pad1)
- U1 pad 3: /TXD -> GND
- U1 pad 4: Net-(M1-Pad5) -> Net-(R3-Pad1)
- U1 pad 5: Net-(M1-Pad45) -> Net-(R2-Pad2)
- U1 pad 6: Net-(M1-Pad45) -> Net-(C1-Pad1)
- U2 pad 3: /RXD -> /TXD
- U2 pad 4: Net-(M1-Pad6) -> Net-(M1-Pad5)
- U2 pad 5: GND -> Net-(M1-Pad45)
- U3 pad 1: Net-(M1-Pad26) -> /VCC_LP
- U3 pad 2: Net-(M1-Pad29) -> GND
- U3 pad 3: Net-(M1-Pad27) -> /RXD
- U3 pad 4: GND -> Net-(M1-Pad6)
- U3 pad 5: Net-(U3-Pad5) -> GND
- U3 pad 6: Net-(M1-Pad28) -> Net-(M1-Pad45)
- U4 pad 1: Net-(M1-Pad27) -> Net-(C6-Pad1)
- U4 pad 2: GND -> Net-(M1-Pad29)
- U4 pad 3: Net-(M1-Pad28) -> Net-(M1-Pad27)
- U4 pad 4: Net-(M1-Pad29) -> GND
- U4 pad 5: Net-(M1-Pad26) -> Net-(U4-Pad5)
- U4 pad 6: Net-(U4-Pad6) -> Net-(M1-Pad28)
- U5 pad 1: Net-(C2-Pad1) -> Net-(C4-Pad1)
- U5 pad 3: Net-(C2-Pad1) -> Net-(C4-Pad1)
- U5 pad 5: Net-(C1-Pad1) -> Net-(C2-Pad1)
- U6 pad 1: GND -> Net-(M1-Pad29)
- U6 pad 2: Net-(C8-Pad1) -> GND
- U6 pad 3: GND -> Net-(M1-Pad28)
- U6 pad 4: Net-(R3-Pad1) -> Net-(M1-Pad27)
- U6 pad 5: Net-(R4-Pad2) -> Net-(C6-Pad1)
- U6 pad 6: Net-(C8-Pad1) -> Net-(U6-Pad6)
Routing:
- net GND: track 0.00 -> 281.2 mm, vias 0 -> 58
- net Net-(C4-Pad1): track 0.00 -> 81.9 mm, vias 0 -> 3
- net /RES: track 0.00 -> 78.2 mm, vias 0 -> 1
- net Net-(C6-Pad1): track 0.00 -> 75.4 mm, vias 0 -> 2
- net /PWR_ON: track 0.00 -> 73.7 mm, vias 0 -> 1
- net Net-(M1-Pad45): track 0.00 -> 66.9 mm, vias 0 -> 3
- net Net-(M1-Pad28): track 0.00 -> 61.6 mm, vias 0 -> 2
- net Net-(M1-Pad27): track 0.00 -> 58.6 mm, vias 0 -> 1
- net Net-(M1-Pad29): track 0.00 -> 47.6 mm, vias 0 -> 1
- net Net-(M1-Pad11): track 0.00 -> 43.9 mm, vias 0 -> 2
- net Net-(C1-Pad1): track 0.00 -> 38.0 mm
- net Net-(M1-Pad1): track 0.00 -> 34.0 mm, vias 0 -> 2
- net /VCC_LP: track 0.00 -> 29.1 mm, vias 0 -> 1
- net Net-(C10-Pad1): track 0.00 -> 27.5 mm
- net /TXD: track 0.00 -> 27.1 mm, vias 0 -> 1
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- added copper zone on B.Cu, net GND
- added copper zone on F.Cu, net GND
- added copper zone on F.Cu, net Net-(C4-Pad1)
Other:
- board outline added: 50 x 70 mm
- net class Default: clearance 0.2 -> 0.23; via_dia 0.6 -> 0.7; via_drill 0.4 -> 0.3
- net class MAIN_PWR added: clearance 0.23, trace_width 1, via_dia 0.7, via_drill 0.3
- net class PWR added: clearance 0.23, trace_width 0.5, via_dia 0.7, via_drill 0.3
- net class PWR2 added: clearance 0.23, trace_width 0.4, via_dia 0.7, via_drill 0.3
- rule trace_clearance: 0.2 -> 0.23

Commit message: Yet another weekly commit
Parts:
- removed P1: CONN_01X06, Pin_Headers:Pin_Header_Angled_1x06
- added C11: 0.1uF, Capacitors_SMD:C_0603, F.Cu at (138.5, 61.0)
- added C12: 0.1uF, Capacitors_SMD:C_0603, F.Cu at (129.5, 61.0)
- added C13: 0.1uF, Capacitors_SMD:C_0603, F.Cu at (132.5, 61.0)
- added C14: 0.1uF, Capacitors_SMD:C_0603, F.Cu at (142.0, 61.0)
- added C15: 0.22uF, Capacitors_SMD:C_0603, F.Cu at (133.0, 68.0)
- added C16: 0.22uF, Capacitors_SMD:C_0603, F.Cu at (137.0, 68.0)
- added D4: ESD7471, Meshium:SOD-882, F.Cu at (136.1, 95.8)
- added R7: 0, Resistors_SMD:R_0603, F.Cu at (135.5, 61.2)
- added R8: 22R, Resistors_SMD:R_0603, F.Cu at (137.0, 70.0)
- added R9: 22R, Resistors_SMD:R_0603, F.Cu at (133.0, 70.0)
- added S5: CONN_01X06, Pin_Headers:Pin_Header_Straight_1x06, B.Cu at (123.0, 52.0)
- added S6: IPEX-20279-001E-01, Meshium:IPEX-20279-001E-01, F.Cu at (137.4, 97.7)
- C6: value 1uF -> 0.1uF
- S1, S2: value CONN_01X10 -> CONN_02X10; footprint Pin_Headers:Pin_Header_Straight_1x10 -> Meshium:Pin_Header_Straight_2x10
- U2, U3: value SN74LVC1T45DBVR -> SN74LVC2T45DCT; footprint Meshium:SOT23-6 -> Meshium:SSOP-8
- moved C7 6.95 mm to (141.0, 52.0), turned to 90 degrees
- moved C2 5.08 mm to (136.0, 57.0), turned to 90 degrees
- moved R1 4.31 mm to (133.0, 57.0), turned to 180 degrees
- moved U3 3.76 mm to (129.4, 63.5)
- moved S2 2.54 mm to (165.5, 72.0)
- moved R5 2.36 mm to (160.0, 91.2)
- moved R6 2.36 mm to (161.7, 91.2)
- moved U2 2.10 mm to (138.5, 63.5)
- moved U5 1.81 mm to (141.0, 58.0)
- moved U6 1.49 mm to (127.0, 56.0)
- moved U1 0.60 mm to (151.5, 58.0)
- moved C6 0.54 mm to (123.0, 58.0)
- moved R3 0.53 mm to (154.0, 52.0)
- moved L1 0.52 mm to (146.5, 63.0)
- moved C3 0.52 mm to (143.0, 52.0)
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Connections:
- M1 pad 167: GND -> (no net)
- M1 pad 168: GND -> (no net)
- M1 pad 169: GND -> (no net)
- M1 pad 170: GND -> (no net)
- M1 pad 171: GND -> (no net)
- M1 pad 172: GND -> (no net)
- M1 pad 173: GND -> (no net)
- M1 pad 174: GND -> (no net)
- M1 pad 175: GND -> (no net)
- M1 pad 176: GND -> (no net)
- M1 pad 177: GND -> (no net)
- M1 pad 178: GND -> (no net)
- M1 pad 179: GND -> (no net)
- M1 pad 180: GND -> (no net)
- M1 pad 181: GND -> (no net)
- M1 pad 182: GND -> (no net)
- M1 pad 183: GND -> (no net)
- M1 pad 184: GND -> (no net)
- M1 pad 185: GND -> (no net)
- M1 pad 186: GND -> (no net)
- M1 pad 187: GND -> (no net)
- M1 pad 188: GND -> (no net)
- M1 pad 189: GND -> (no net)
- M1 pad 190: GND -> (no net)
- M1 pad 191: GND -> (no net)
- M1 pad 192: GND -> (no net)
- M1 pad 193: GND -> (no net)
- M1 pad 194: GND -> (no net)
- M1 pad 195: GND -> (no net)
- M1 pad 196: GND -> (no net)
- M1 pad 197: GND -> (no net)
- M1 pad 198: GND -> (no net)
- M1 pad 199: GND -> (no net)
- M1 pad 200: GND -> (no net)
- M1 pad 201: GND -> (no net)
- M1 pad 202: GND -> (no net)
- M1 pad 203: GND -> (no net)
- M1 pad 204: GND -> (no net)
- M1 pad 205: GND -> (no net)
- M1 pad 206: GND -> (no net)
- M1 pad 207: GND -> (no net)
- M1 pad 208: GND -> (no net)
- M1 pad 209: GND -> (no net)
- M1 pad 210: GND -> (no net)
- M1 pad 211: GND -> (no net)
- M1 pad 212: GND -> (no net)
- M1 pad 213: GND -> (no net)
- M1 pad 214: GND -> (no net)
- M1 pad 215: GND -> (no net)
- M1 pad 216: GND -> (no net)
- M1 pad 217: GND -> (no net)
- M1 pad 218: GND -> (no net)
- M1 pad 219: GND -> (no net)
- M1 pad 220: GND -> (no net)
- M1 pad 221: GND -> (no net)
- M1 pad 222: GND -> (no net)
- M1 pad 223: GND -> (no net)
- M1 pad 224: GND -> (no net)
- M1 pad 225: GND -> (no net)
- M1 pad 226: GND -> (no net)
- M1 pad 227: GND -> (no net)
- M1 pad 228: GND -> (no net)
- M1 pad 229: GND -> (no net)
- M1 pad 230: GND -> (no net)
- M1 pad 231: GND -> (no net)
- M1 pad 232: GND -> (no net)
- M1 pad 233: GND -> (no net)
- M1 pad 234: GND -> (no net)
- M1 pad 235: (no net) -> Net-(M1-Pad235)
- M1 pad 4: Net-(M1-Pad3) -> Net-(M1-Pad4)
- M1 pad 45: Net-(M1-Pad45) -> Net-(C13-Pad1)
- M1 pad 66: Net-(M1-Pad66) -> SIM_SEL
- Q1 pad 2: /PWR_ON -> PWR_ON
- Q1 pad 5: /RES -> RES
- R1 pad 2: /VCC_LP -> Net-(C11-Pad1)
- S1 pad 1: /VCC_LP -> Net-(C11-Pad1)
- S1 pad 2: Net-(S1-Pad2) -> Net-(M1-Pad16)
- S1 pad 3: /RXD -> Net-(S1-Pad3)
- S1 pad 4: /TXD -> GND
- S1 pad 5: /PWR_ON -> RXD
- S1 pad 6: /RES -> Net-(R8-Pad2)
- S1 pad 7: Net-(S1-Pad7) -> TXD
- S1 pad 9: Net-(S1-Pad9) -> PWR_ON
- S2 pad 1: GND -> Net-(S2-Pad1)
- S2 pad 2: Net-(S2-Pad2) -> GND
- S2 pad 7: Net-(S2-Pad7) -> RTS
- S2 pad 9: Net-(S2-Pad9) -> CTS
- U2 pad 1: /VCC_LP -> Net-(C11-Pad1)
- U2 pad 2: GND -> RTS
- U2 pad 3: /TXD -> TXD
- U2 pad 4: Net-(M1-Pad5) -> GND
- U2 pad 5: Net-(M1-Pad45) -> Net-(C11-Pad1)
- U2 pad 6: Net-(M1-Pad45) -> Net-(M1-Pad5)
- U3 pad 1: /VCC_LP -> Net-(C11-Pad1)
- U3 pad 2: GND -> CTS
- U3 pad 3: /RXD -> RXD
- U3 pad 4: Net-(M1-Pad6) -> GND
- U3 pad 6: Net-(M1-Pad45) -> Net-(M1-Pad6)
Routing:
- net GND: track 281.2 -> 13.0 mm, vias 58 -> 4
- net RES: track 0.00 -> 79.0 mm, vias 0 -> 1
- net /RES: track 78.2 -> 0.00 mm, vias 1 -> 0
- net /PWR_ON: track 73.7 -> 0.00 mm, vias 1 -> 0
- net PWR_ON: track 0.00 -> 73.4 mm, vias 0 -> 1
- net Net-(M1-Pad45): track 66.9 -> 0.00 mm, vias 3 -> 0
- net Net-(C6-Pad1): track 75.4 -> 19.8 mm, vias 2 -> 1
- net Net-(M1-Pad28): track 61.6 -> 6.32 mm, vias 2 -> 0
- net CTS: track 0.00 -> 55.3 mm, vias 0 -> 1
- net Net-(M1-Pad27): track 58.6 -> 6.48 mm, vias 1 -> 0
- net Net-(M1-Pad29): track 47.6 -> 7.14 mm, vias 1 -> 0
- net /VCC_LP: track 29.1 -> 0.00 mm, vias 1 -> 0
- net TXD: track 0.00 -> 28.6 mm, vias 0 -> 1
- net /TXD: track 27.1 -> 0.00 mm, vias 1 -> 0
- net Net-(C13-Pad1): track 0.00 -> 24.7 mm
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
Commit message: Weekly commit
Parts:
- removed C11, C12, C13, C14: 0.1uF, Capacitors_SMD:C_0603
- moved R7 27.5 mm to (161.1, 71.4), turned to 0 degrees
- moved C15 5.43 mm to (138.4, 67.3), turned to 0 degrees
- moved C6 5.31 mm to (128.0, 59.8), turned to 0 degrees
- moved U6 4.47 mm to (131.0, 58.0), turned to 180 degrees
- moved Q1 3.00 mm to (158.0, 85.0)
- moved Q2 3.00 mm to (158.0, 88.0)
- moved U2 2.14 mm to (137.0, 62.0)
- moved R9 1.96 mm to (134.3, 68.5), turned to 90 degrees
- moved R8 1.83 mm to (135.9, 68.5), turned to 90 degrees
- moved U3 1.75 mm to (128.5, 62.0)
- moved C16 1.65 mm to (138.4, 68.9), turned to 0 degrees
- moved R1 1.60 mm to (133.6, 58.5), turned to 270 degrees
- moved D1 0.98 mm to (167.0, 102.0)
- moved R6 0.87 mm to (162.0, 92.0)
- moved R5 0.82 mm to (160.0, 92.0)
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Connections:
- M1 pad 45: Net-(C13-Pad1) -> Net-(M1-Pad45)
- Q1 pad 2: PWR_ON -> Net-(M1-Pad1)
- Q1 pad 3: Net-(M1-Pad11) -> Net-(Q1-Pad3)
- Q1 pad 5: RES -> Net-(M1-Pad60)
- Q1 pad 6: Net-(M1-Pad59) -> Net-(Q1-Pad6)
- Q2 pad 1: Net-(Q2-Pad1) -> GND
- Q2 pad 2: Net-(M1-Pad1) -> PWR_ON
- Q2 pad 3: Net-(Q2-Pad3) -> Net-(M1-Pad11)
- Q2 pad 5: Net-(M1-Pad60) -> RES
- Q2 pad 6: GND -> Net-(M1-Pad59)
- R5 pad 2: Net-(Q2-Pad1) -> Net-(Q1-Pad6)
- R6 pad 2: Net-(Q2-Pad3) -> Net-(Q1-Pad3)
- S5 pad 2: Net-(M1-Pad27) -> Net-(M1-Pad29)
- S5 pad 3: Net-(M1-Pad29) -> Net-(M1-Pad28)
- S5 pad 4: Net-(M1-Pad28) -> Net-(M1-Pad27)
- U2 pad 8: Net-(C13-Pad1) -> Net-(M1-Pad45)
- U3 pad 8: Net-(C13-Pad1) -> Net-(U3-Pad8)
- U6 pad 1: Net-(M1-Pad29) -> Net-(U6-Pad1)
- U6 pad 6: Net-(U6-Pad6) -> Net-(M1-Pad29)
Routing:
- net Net-(M1-Pad28): track 6.32 -> 74.2 mm, vias 0 -> 1
- net Net-(M1-Pad27): track 6.48 -> 60.4 mm
- net Net-(M1-Pad29): track 7.14 -> 60.0 mm, vias 0 -> 1
- net Net-(M1-Pad45): track 0.00 -> 45.4 mm, vias 0 -> 2
- net SIM_SEL: track 0.00 -> 44.2 mm, vias 0 -> 1
- net Net-(C6-Pad1): track 19.8 -> 54.5 mm
- net CTS: track 55.3 -> 30.1 mm
- net Net-(C13-Pad1): track 24.7 -> 0.00 mm
- net Net-(C4-Pad1): track 87.8 -> 63.2 mm, vias 2 -> 3
- net Net-(M1-Pad4): track 24.4 -> 0.00 mm, vias 2 -> 0
- net TXD: track 28.6 -> 5.04 mm, vias 1 -> 0
- net Net-(R8-Pad2): track 24.2 -> 1.71 mm, vias 1 -> 0
- net Net-(M1-Pad16): track 0.00 -> 22.0 mm, vias 0 -> 1
- net Net-(M1-Pad6): track 20.5 -> 0.00 mm
- net RES: track 79.0 -> 60.1 mm
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- removed copper zone on F.Cu, net Net-(C4-Pad1)

Commit message: PCB tracerouting
Parts:
- moved C15 6.01 mm to (132.5, 68.5), turned to 90 degrees
- moved C6 2.22 mm to (126.4, 58.3), turned to 270 degrees
- moved R1 1.18 mm to (133.8, 59.6)
- moved C7 1.00 mm to (140.0, 52.0)
- moved U2 1.00 mm to (138.0, 62.0)
- moved U6 0.50 mm to (131.0, 57.5)
Connections:
- U3 pad 8: Net-(U3-Pad8) -> Net-(M1-Pad45)
Routing:
- net GND: track 14.0 -> 74.2 mm, vias 7 -> 11
- net Net-(M1-Pad45): track 45.4 -> 82.9 mm, vias 2 -> 4
- net Net-(M1-Pad4): track 0.00 -> 31.5 mm, vias 0 -> 2
- net Net-(M1-Pad6): track 0.00 -> 31.4 mm, vias 0 -> 2
- net Net-(R1-Pad2): track 6.29 -> 36.3 mm, vias 0 -> 2
- net CTS: track 30.1 -> 59.7 mm, vias 1 -> 2
- net TXD: track 5.04 -> 27.6 mm, vias 0 -> 1
- net Net-(R8-Pad2): track 1.71 -> 22.8 mm, vias 0 -> 1
- net RTS: track 29.3 -> 49.7 mm, vias 1 -> 2
- net RXD: track 0.06 -> 20.4 mm, vias 0 -> 1
- net Net-(C15-Pad1): track 0.00 -> 11.0 mm
- net Net-(M1-Pad3): track 5.52 -> 16.5 mm
- net Net-(R9-Pad2): track 10.9 -> 21.8 mm, vias 0 -> 1
- net Net-(M1-Pad5): track 5.51 -> 15.7 mm
- net Net-(C16-Pad1): track 0.00 -> 9.57 mm
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
Commit message: PCB tracerouting
Parts:
- moved D3 2.11 mm to (153.5, 98.3), turned to 180 degrees
- moved D1 2.00 mm to (167.0, 100.0), turned to 0 degrees
- moved D2 2.00 mm to (167.0, 102.0), turned to 0 degrees
- moved S4 1.25 mm to (155.2, 96.9)
- moved D4 0.85 mm to (136.9, 96.2)
- moved A1 0.40 mm to (146.4, 118.0)
- moved S6 0.31 mm to (137.5, 98.0)
- moved J2 0.23 mm to (146.4, 96.9)
Connections:
- M1 pad 167: (no net) -> GND
- M1 pad 168: (no net) -> GND
- M1 pad 169: (no net) -> GND
- M1 pad 170: (no net) -> GND
Routing:
- net Net-(C4-Pad1): track 64.2 -> 106.8 mm, vias 3 -> 4
- net GND: track 74.2 -> 115.5 mm, vias 11 -> 13
- net Net-(D4-Pad1): track 0.00 -> 9.23 mm
- net Net-(J2-Pad1): track 0.07 -> 7.77 mm
- net Net-(D2-Pad2): track 9.94 -> 15.4 mm
- net (no net): track 8.83 -> 3.94 mm
- net Net-(D3-Pad2): track 9.47 -> 8.13 mm
